File: untitled.sch (EAGLE design)
At the start: 68 parts, among them J1 5V, J2 R1171S421B-E2-FE, Q1 2N7002KW, Q10 2N7002KW, Q11 BSS138LT3G, Q2 2N7002KW, Q8 DMP2035U-7, Q9 2N7002KW, SW1 B3U-1000P-2P-SMD, SW2 B3U-1000P-2P-SMD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

Commit message: ver1.0
Parts:
- added C23: 10uf, Seeed-Capacitor:CERAMIC-10UF-10V-10%-X5R(0603)
- added SW4: B3U-1000P-2P-SMD, Seeed-Switch:SMD-BUTTON(2P-3.0X2.5X1.2+0.4MM)-B3U-1000P-2P-SMD
- added U$31: 10K, Seeed-Resistor:SMD-RES-10K-5%-1/(0402)
Connections:
- removed net ANT_POWR: U2.IO19
- new net TRAP_FORCE: C23.1, SW4.1, U$31.2, U2.IO35
- net GND: now also C23.2, U$31.1
- net PWRKEY: no longer JP1.13
- net RESET_N: no longer JP1.12
- net RXD_MODULE: now also U9.A3; no longer U9.A4
- net RX_MODULE2: now also JP1.4, U9.B3; no longer JP1.5, U9.B4
- net TXD_MODULE: now also U9.A4; no longer U9.A3
- net TX_MODULE2: now also JP1.5, U9.B4; no longer JP1.4, U9.B3
- net VDD_1V8: no longer JP1.11
- net VDD_3V3: now also SW4.2; no longer JP1.10

Commit message: MOSをSeeedのものに変更
Parts:
- Q1, Q10, Q2, Q9: value 2N7002KW -> BSS138W-7-F; device Discrete-new:MOSFET-N+'SI1304BDL' -> Seeed-Transistor:SMD-MOSFET-N-CH-50V-200MA-BSS138W-7-F(SOT-23)
- Q11: value BSS138LT3G -> CJ2302; device Discrete-new:MOSFET-N+'SOT23' -> Seeed-Transistor:SMD-MOSFET-N-CH-20V-2.1A-CJ2302(SOT-23)
- Q8: value DMP2035U-7 -> NCE3407A; device Discrete-new:MOSFET-P'SI2323CDS/SI2305DS<BR>' -> Seeed-Transistor:SMD-MOSFET-P-CH-VDC=30V-ID=4.3A-NCE3407A(SOT-23)
Connections:
- net BATTERY_CHECK: now also JP1.8
- net RX_ESP: now also JP1.9; no longer JP1.8
- net TX_ESP: now also JP1.10; no longer JP1.9
